File: display/pcb/ws2812matrix_leds.sch (KiCad schematic (older format))
At the start: 174 parts, among them M201 CC_MOUNT, M202 CC_MOUNT, M203 CC_MOUNT, Q201 MOS_N, U201 CC_WS2812B, U202 CC_WS2812B, U203 CC_WS2812B, U204 CC_WS2812B, U205 CC_WS2812B, U206 CC_WS2812B, U207 CC_WS2812B, U208 CC_WS2812B, U209 CC_WS2812B, U210 CC_WS2812B, U211 CC_WS2812B, U212 CC_WS2812B, U213 CC_WS2812B, U214 CC_WS2812B, U215 CC_WS2812B, U216 CC_WS2812B, U217 CC_WS2812B, U218 CC_WS2812B, U219 CC_WS2812B, U220 CC_WS2812B, U221 CC_WS2812B, U222 CC_WS2812B, U223 CC_WS2812B, U224 CC_WS2812B, U225 CC_WS2812B, U226 CC_WS2812B, U227 CC_WS2812B, U228 CC_WS2812B, U229 CC_WS2812B, U230 CC_WS2812B, U231 CC_WS2812B, U232 CC_WS2812B, U233 CC_WS2812B, U234 CC_WS2812B, U235 CC_WS2812B, U236 CC_WS2812B, U237 CC_WS2812B, U238 CC_WS2812B, U239 CC_WS2812B, U240 CC_WS2812B, U241 CC_WS2812B, U242 CC_WS2812B, U243 CC_WS2812B, U244 CC_WS2812B, U245 CC_WS2812B, U246 CC_WS2812B, U247 CC_WS2812B, U248 CC_WS2812B, U249 CC_WS2812B, U250 CC_WS2812B, U251 CC_WS2812B, U252 CC_WS2812B, U253 CC_WS2812B, U254 CC_WS2812B, U255 CC_WS2812B, U256 CC_WS2812B, U257 CC_WS2812B, U258 CC_WS2812B, U259 CC_WS2812B, U260 CC_WS2812B, U261 CC_WS2812B, U262 CC_WS2812B, U263 CC_WS2812B, U264 CC_WS2812B, U265 CC_WS2812B, U266 CC_WS2812B, U267 CC_WS2812B, U268 CC_WS2812B, U269 CC_WS2812B, U270 CC_WS2812B, U271 CC_WS2812B, U272 CC_WS2812B, U273 CC_WS2812B, U274 CC_WS2812B, U275 CC_WS2812B, U276 CC_WS2812B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

Commit message: fixed license statements for svg and kicad files
Parts:
- U201, U202, U203, U204, U205, U206, U207, U208, U209, U210, U211, U212, U213, U214, U215, U216, U217, U218, U219, U220, U221, U222, U223, U224, U225, U226, U227, U228, U229, U230, U231, U232, U233, U234, U235, U236, U237, U238, U239, U240, U241, U242, U243, U244, U245, U246, U247, U248, U249, U250, U251, U252, U253, U254, U255, U256, U257, U258, U259, U260, U261, U262, U263, U264, U265, U266, U267, U268, U269, U270, U271, U272, U273, U274, U275, U276, U277, U278, U279, U280, U281, U282, U283, U284: symbol CC_WS2812B -> CC_WS2812B-RESCUE-ws2812display
