File: display/pcb.v2/ws2812display.kicad_pcb (KiCad board)
At the start: 2 copper layers, 100 x 100 mm, 88 parts, among them J101 USB-MINIB, M201 CC_MOUNT, M202 CC_MOUNT, M203 CC_MOUNT, M204 CC_MOUNT, P102 CONN_01X02, P103 CONN_01X02, P104 CONN_01X02, P105 CONN_01X02, P106 CONN_01X02, P107 CONN_01X02, P108 CONN_01X03, P110 CONN_01X02, Q201 MOS_N, SW101 SW_PUSH, SW102 SW_PUSH, U101 CC_XC6204, U102 CC_STM32F401xE, U104 CC_STM32SWD, U265 CC_WS2812B, U266 CC_WS2812B, U267 CC_WS2812B, U268 CC_WS2812B, U269 CC_WS2812B, U270 CC_WS2812B, U271 CC_WS2812B, U272 CC_WS2812B, U273 CC_WS2812B, U274 CC_WS2812B, U275 CC_WS2812B, U276 CC_WS2812B, U277 CC_WS2812B, U278 CC_WS2812B, U279 CC_WS2812B, U280 CC_WS2812B, U281 CC_WS2812B, U282 CC_WS2812B, U283 CC_WS2812B, U284 CC_WS2812B, X101 12MHz

Commit message: final pcb design for v2
Parts:
- added U1: CC_WS2812B, cc_display:WS2812B, B.Cu at (96.0, 55.0)
- added U10: CC_WS2812B, cc_display:WS2812B, B.Cu at (55.0, 84.0)
- added U11: CC_WS2812B, cc_display:WS2812B, B.Cu at (125.0, 96.0)
- added U12: CC_WS2812B, cc_display:WS2812B, B.Cu at (113.0, 96.0)
- added U13: CC_WS2812B, cc_display:WS2812B, B.Cu at (96.0, 96.0)
- added U14: CC_WS2812B, cc_display:WS2812B, B.Cu at (84.0, 96.0)
- added U15: CC_WS2812B, cc_display:WS2812B, B.Cu at (67.0, 96.0)
- added U16: CC_WS2812B, cc_display:WS2812B, B.Cu at (55.0, 96.0)
- added U17: CC_WS2812B, cc_display:WS2812B, B.Cu at (100.0, 113.0)
- added U18: CC_WS2812B, cc_display:WS2812B, B.Cu at (80.0, 113.0)
- added U19: CC_WS2812B, cc_display:WS2812B, B.Cu at (100.0, 125.0)
- added U2: CC_WS2812B, cc_display:WS2812B, B.Cu at (84.0, 55.0)
- added U20: CC_WS2812B, cc_display:WS2812B, B.Cu at (80.0, 125.0)
- added U3: CC_WS2812B, cc_display:WS2812B, B.Cu at (96.0, 67.0)
- added U4: CC_WS2812B, cc_display:WS2812B, B.Cu at (84.0, 67.0)
- added U5: CC_WS2812B, cc_display:WS2812B, B.Cu at (125.0, 84.0)
- added U6: CC_WS2812B, cc_display:WS2812B, B.Cu at (113.0, 84.0)
- added U7: CC_WS2812B, cc_display:WS2812B, B.Cu at (96.0, 84.0)
- added U8: CC_WS2812B, cc_display:WS2812B, B.Cu at (84.0, 84.0)
- added U9: CC_WS2812B, cc_display:WS2812B, B.Cu at (67.0, 84.0)
Connections:
- net Net-(U265-Pad2) renamed /LEDS/D5
- net Net-(U265-Pad4) renamed /LEDS/D4
- net Net-(U266-Pad2) renamed /LEDS/D11
- net Net-(U266-Pad4) renamed /LEDS/D10
- net Net-(U267-Pad2) renamed /LEDS/D6
- net Net-(U268-Pad2) renamed /LEDS/D12
- net Net-(U269-Pad2) renamed /LEDS/D1
- net Net-(U270-Pad2) renamed /LEDS/D3
- net Net-(U270-Pad4) renamed /LEDS/D2
- net Net-(U271-Pad2) renamed /LEDS/D7
- net Net-(U272-Pad2) renamed /LEDS/D13
- net Net-(U273-Pad2) renamed /LEDS/D17
- net Net-(U273-Pad4) renamed /LEDS/D16
- net Net-(U274-Pad2) renamed /LEDS/D19
- net Net-(U274-Pad4) renamed /LEDS/D18
- net Net-(U277-Pad2) renamed /LEDS/D8
- net Net-(U278-Pad2) renamed /LEDS/D14
- net Net-(U281-Pad2) renamed /LEDS/D9
- net Net-(U282-Pad2) renamed /LEDS/D15
- U101 pad 4: (no net) -> Net-(U101-Pad4)
- U102 pad 10: (no net) -> Net-(U102-Pad10)
- U102 pad 11: (no net) -> Net-(U102-Pad11)
- U102 pad 14: (no net) -> Net-(U102-Pad14)
- U102 pad 15: (no net) -> Net-(U102-Pad15)
- U102 pad 20: (no net) -> Net-(U102-Pad20)
- U102 pad 24: (no net) -> Net-(U102-Pad24)
- U102 pad 25: (no net) -> Net-(U102-Pad25)
- U102 pad 28: (no net) -> Net-(U102-Pad28)
- U102 pad 29: (no net) -> Net-(U102-Pad29)
- U102 pad 3: (no net) -> Net-(U102-Pad3)
- U102 pad 33: (no net) -> Net-(U102-Pad33)
- U102 pad 34: (no net) -> Net-(U102-Pad34)
- U102 pad 35: (no net) -> Net-(U102-Pad35)
- U102 pad 36: (no net) -> Net-(U102-Pad36)
- U102 pad 37: (no net) -> Net-(U102-Pad37)
- U102 pad 38: (no net) -> Net-(U102-Pad38)
- U102 pad 39: (no net) -> Net-(U102-Pad39)
- U102 pad 4: (no net) -> Net-(U102-Pad4)
- U102 pad 40: (no net) -> Net-(U102-Pad40)
- U102 pad 41: (no net) -> Net-(U102-Pad41)
- U102 pad 50: (no net) -> Net-(U102-Pad50)
- U102 pad 54: (no net) -> Net-(U102-Pad54)
- U102 pad 58: (no net) -> Net-(U102-Pad58)
- U102 pad 59: (no net) -> Net-(U102-Pad59)
- U102 pad 61: (no net) -> Net-(U102-Pad61)
- U102 pad 62: (no net) -> Net-(U102-Pad62)
- U102 pad 8: (no net) -> Net-(U102-Pad8)
- U102 pad 9: (no net) -> Net-(U102-Pad9)
Other:
- board text added: "CC 20160725 rev. 2"
- board text removed: "CC 20151102 rev. 0"
