File: display/pcb.v2/ws2812matrix_leds.sch (KiCad schematic (older format))
At the start: 47 parts, among them M201 CC_MOUNT, M202 CC_MOUNT, M203 CC_MOUNT, M204 CC_MOUNT, Q201 MOS_N, U265 CC_WS2812B, U266 CC_WS2812B, U267 CC_WS2812B, U268 CC_WS2812B, U269 CC_WS2812B, U270 CC_WS2812B, U271 CC_WS2812B, U272 CC_WS2812B, U273 CC_WS2812B, U274 CC_WS2812B, U275 CC_WS2812B, U276 CC_WS2812B, U277 CC_WS2812B, U278 CC_WS2812B, U279 CC_WS2812B, U280 CC_WS2812B, U281 CC_WS2812B, U282 CC_WS2812B, U283 CC_WS2812B, U284 CC_WS2812B

Commit message: final pcb design for v2
Parts:
- added U1, U10, U11, U12, U13, U14, U15, U16, U17, U18, U19, U2, U20, U3, U4, U5, U6, U7, U8, U9: CC_WS2812B, cc_display:WS2812B, symbol CC_WS2812B
Connections:
- net DIN_IN: now also U1.4 (DIN)
- net GND: now also U1.3 (VSS), U10.3 (VSS), U11.3 (VSS), U12.3 (VSS), U13.3 (VSS), U14.3 (VSS), U15.3 (VSS), U16.3 (VSS), U17.3 (VSS), U18.3 (VSS), U19.3 (VSS), U2.3 (VSS), U20.3 (VSS), U3.3 (VSS), U4.3 (VSS), U5.3 (VSS), U6.3 (VSS), U7.3 (VSS), U8.3 (VSS), U9.3 (VSS)
- net MATRIX_DOUT: now also U20.2 (DOUT)
- net VCC: now also U1.1 (VDD), U10.1 (VDD), U11.1 (VDD), U12.1 (VDD), U13.1 (VDD), U14.1 (VDD), U15.1 (VDD), U16.1 (VDD), U17.1 (VDD), U18.1 (VDD), U19.1 (VDD), U2.1 (VDD), U20.1 (VDD), U3.1 (VDD), U4.1 (VDD), U5.1 (VDD), U6.1 (VDD), U7.1 (VDD), U8.1 (VDD), U9.1 (VDD)
- net D1: now reaches U269.2 (DOUT), U275.4 (DIN)
- net D1: now also U1.2 (DOUT), U2.4 (DIN)
- net D2: now reaches U270.4 (DIN), U275.2 (DOUT)
- net D2: now also U2.2 (DOUT), U3.4 (DIN)
- net D3: now reaches U270.2 (DOUT), U276.4 (DIN)
- net D3: now also U3.2 (DOUT), U4.4 (DIN)
- net D4: now reaches U265.4 (DIN), U276.2 (DOUT)
- net D4: now also U4.2 (DOUT), U5.4 (DIN)
- net D7: now reaches U271.2 (DOUT), U277.4 (DIN)
- net D7: now also U7.2 (DOUT), U8.4 (DIN)
- net D6: now reaches U267.2 (DOUT), U271.4 (DIN)
- net D6: now also U6.2 (DOUT), U7.4 (DIN)
- net D8: now reaches U277.2 (DOUT), U281.4 (DIN)
- net D8: now also U8.2 (DOUT), U9.4 (DIN)
- net D5: now reaches U265.2 (DOUT), U267.4 (DIN)
- net D5: now also U5.2 (DOUT), U6.4 (DIN)
- net D10: now reaches U266.4 (DIN), U283.2 (DOUT)
- net D10: now also U10.2 (DOUT), U11.4 (DIN)
- net D9: now reaches U281.2 (DOUT), U283.4 (DIN)
- net D9: now also U10.4 (DIN), U9.2 (DOUT)
- net D13: now reaches U272.2 (DOUT), U278.4 (DIN)
- net D13: now also U13.2 (DOUT), U14.4 (DIN)
- net D12: now reaches U268.2 (DOUT), U272.4 (DIN)
- net D12: now also U12.2 (DOUT), U13.4 (DIN)
- net D11: now reaches U266.2 (DOUT), U268.4 (DIN)
- net D11: now also U11.2 (DOUT), U12.4 (DIN)
- net D16: now reaches U273.4 (DIN), U284.2 (DOUT)
- net D16: now also U16.2 (DOUT), U17.4 (DIN)
- net D15: now reaches U282.2 (DOUT), U284.4 (DIN)
- net D15: now also U15.2 (DOUT), U16.4 (DIN)
- net D14: now reaches U278.2 (DOUT), U282.4 (DIN)
- net D14: now also U14.2 (DOUT), U15.4 (DIN)
- net D17: now reaches U273.2 (DOUT), U279.4 (DIN)
- net D17: now also U17.2 (DOUT), U18.4 (DIN)
- net D18: now reaches U274.4 (DIN), U279.2 (DOUT)
- net D18: now also U18.2 (DOUT), U19.4 (DIN)
- net D19: now reaches U274.2 (DOUT), U280.4 (DIN)
- net D19: now also U19.2 (DOUT), U20.4 (DIN)
